File: hardware/rev2_secure-edge-logger/ESP32-C3-02.kicad_sch (KiCad schematic)
At the start: 30 parts, among them J3 GSD090012SEU, U2 CP2102N-Axx-xQFN20, U3 ESP32-C3-WROOM-02-H4, U4 W25Q32JVSSIQ, U5 USBLC6-2SC6

Commit message: Add files via upload
Parts:
- removed U2: CP2102N-Axx-xQFN20, Package_DFN_QFN:SiliconLabs_QFN-20-1EP_3x3mm_P0.5mm_EP1.8x1.8mm, symbol Interface_USB:CP2102N-Axx-xQFN20
- added R210, R211, R212, R213, R214: 10k, Resistor_SMD:R_0805_2012Metric, symbol Device:R
- added U200: CP2102N-Axx-xQFN24, Package_DFN_QFN:QFN-24-1EP_4x4mm_P0.5mm_EP2.6x2.6mm, symbol Interface_USB:CP2102N-Axx-xQFN24
- C200: renamed from C10; footprint ESP32Footprints:T491A -> Capacitor_SMD:C_0805_2012Metric
- C204: renamed from C12; value 0.1U -> 0.1u
- C205: renamed from C13; value 1Ou -> 10u; footprint ESP32Footprints:T491A -> Capacitor_SMD:C_1206_3216Metric
- C206: renamed from C15; footprint ESP32Footprints:T491A -> Capacitor_SMD:C_1206_3216Metric
- U203: renamed from U3; footprint ESP32Footprints:MODULE_ESP32-C3-WROOM-02-H4 -> ESP32Footprints:ESP32--C3-WROOM-02-H4
- renumbered C9 to C201, C11 to C202, C16 to C203, C14 to C207, J3 to J200, R1 to R200, R13 to R201, R14 to R202, R12 to R203, R11 to R204, R18 to R205, R15 to R206, R16 to R207, R17 to R208, R30 to R209, RX1 to RX200, TX1 to TX200, U5 to U201, U4 to U202
Connections:
- net +3.3V: now also C200.1, R210.2, R211.2, R212.2, R213.2, R214.2, U200.5 (VIO), U200.6 (VDD), U200.7 (VREGIN); no longer C200.2
- net CS: now also R214.1
- net CS-SD: now also U203.7 (IO8); no longer U203.4 (IO5)
- net GND: now also C200.2, U200.2 (GND), U200.25 (GND); no longer C200.1, J200.8 (DAT1), J200.9 (DAT2)
- net INT/SQW: now also U203.4 (IO5); no longer U203.7 (IO8)
- net MOSI-DI: now also R210.1
- net RTS: now also U200.19 (~{RTS})
- net RX-TX: now also U200.20 (RXD)
- net TX-RX: now also U200.21 (TXD)
- net USB_D+: now also U200.3 (D+)
- net USB_D-: now also U200.4 (D-)
- net VBUS-CP: now reaches C202.2, R201.1, R202.2
- net VBUS-CP: now also U200.8 (VBUS)
- net MISO-GSD: now reaches J200.7 (DAT0), R208.1
- net MISO-GSD: now also R211.1
- net SCLK-ESP: now reaches R206.2, U203.5 (IO6)
- net MISO-ESP: now reaches R207.1, U203.6 (IO7)
- net MISO-W25: now reaches R205.1, U202.2 (DO(IO1))
- net NRXT: now reaches R204.1
- net NRXT: now also U200.13 (~{RXT}/GPIO.1)
- net NTXT: now reaches R203.1
- net NTXT: now also U200.14 (~{TXT}/GPIO.0)
- net NRST: now reaches R200.2
- net NRST: now also U200.9 (~{RST})
- new net DAT1: J200.8 (DAT1), R212.1
- new net DAT2: J200.9 (DAT2), R213.1
- new net DTR: U200.23 (~{DTR})
- no-connect marks 7 -> 10
Other:
- sheet USER INTERFACE ports: added DTR; removed DTS
- moved on the sheet: C200, C201, C204, C206, C207, J200, R203, R204, R205, R206, R207, R208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
